File: Hardware/Production/SparkFun_MicroMod_Function_ADIN1110-Panel_v01d.brd (EAGLE design)
At the start: 128.7 x 91.4 mm, 345 parts, among them J1 T1_INDUSTRIAL, J2 MICROMOD_FUNCTION_STANDARD, J3 MICROMOD_FUNCTION_STANDARD, J4 T1_INDUSTRIAL, J5 MICROMOD_FUNCTION_STANDARD, J6 T1_INDUSTRIAL, Q1 220mA/50V/3.5Ω, Q2 20V/4.2A/52mΩ/1.4W, Q3 20V/4.2A/52mΩ/1.4W, Q4 220mA/50V/3.5Ω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

Commit message: Update PROD_IDs for 10ohm and 4.7ohm resistors on production panel
Parts:
- R3, R4, R46, R47, R71, R72: value 5.1Ω -> 4.7Ω
- R44, R45, R5, R6, R69, R70: value 10.2Ω -> 10Ω
Changed lines of the file:
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@@
 <attribute name="VALUE" x="28.575040625" y="63.0764" size="0.6096" layer="27" font="vector" ratio="20" rot="R90" align="top-center"/>
 </element>
-<element name="R5" library="SparkFun-Resistors" package="0402-TIGHT" value="10.2Ω" x="20.812759375" y="39.8145" smashed="yes">
+<element name="R5" library="SparkFun-Resistors" package="0402-TIGHT" value="10Ω" x="20.812759375" y="39.8145" smashed="yes">
 <attribute name="NAME" x="20.812759375" y="40.3765" size="0.6096" layer="25" font="vector" ratio="20" align="bottom-center"/>
+<attribute name="PROD_ID" value="RES-16072" x="20.812759375" y="39.8145" size="1.778" layer="27" font="vector" ratio="15" display="off"/>
 <attribute name="VALUE" x="22.89301875" y="40.1542" size="0.6096" layer="27" font="vector" ratio="20" align="top-center"/>
 </element>
-<element name="R6" library="SparkFun-Resistors" package="0402-TIGHT" value="10.2Ω" x="20.289521875" y="38.89501875" smashed="yes">
+<element name="R6" library="SparkFun-Resistors" package="0402-TIGHT" value="10Ω" x="20.289521875" y="38.89501875" smashed="yes">
 <attribute name="NAME" x="20.289521875" y="39.45701875" size="0.6096" layer="25" font="vector" ratio="20" align="bottom-center"/>
+<attribute name="PROD_ID" value="RES-16072" x="20.289521875" y="38.89501875" size="1.778" layer="27" font="vector" ratio="15" display="off"/>
 <attribute name="VALUE" x="22.308821875" y="39.1661375" size="0.6096" layer="27" font="vector" ratio="20" align="top-center"/>
 </element>
-<element name="R4" library="SparkFun-Resistors" package="0402-TIGHT" value="5.1Ω" x="22.501859375" y="42.4459375" smashed="yes" rot="R180">
+<element name="R4" library="SparkFun-Resistors" package="0402-TIGHT" value="4.7Ω" x="22.501859375" y="42.4459375" smashed="yes" rot="R180">
 <attribute name="NAME" x="22.501859375" y="41.8839375" size="0.6096" layer="25" font="vector" ratio="20" rot="R180" align="bottom-center"/>
+<attribute name="PROD_ID" value="RES-16312" x="22.501859375" y="42.4459375" size="1.778" layer="27" font="vector" ratio="15" rot="R180" display="off"/>
 <attribute name="VALUE" x="24.462740625" y="42.1697375" size="0.6096" layer="27" font="vector" ratio="20" rot="R180" align="top-center"/>
 </element>
-<element name="R3" library="SparkFun-Resistors" package="0402-TIGHT" value="5.1Ω" x="18.54961875" y="42.420540625" smashed="yes" rot="R180">
+<element name="R3" library="SparkFun-Resistors" package="0402-TIGHT" value="4.7Ω" x="18.54961875" y="42.420540625" smashed="yes" rot="R180">
 <attribute name="NAME" x="18.54961875" y="41.858540625" size="0.6096" layer="25" font="vector" ratio="20" rot="R180" align="bottom-center"/>
+<attribute name="PROD_ID" value="RES-16312" x="18.54961875" y="42.420540625" size="1.778" layer="27" font="vector" ratio="15" rot="R180" display="off"/>
 <attribute name="VALUE" x="16.624296875" y="42.1672" size="0.6096" layer="27" font="vector" ratio="20" rot="R180" align="top-center"/>
 </element>
@@
 <attribute name="VALUE" x="67.08398125" y="63.0764" size="0.6096" layer="27" font="vector" ratio="20" rot="R90" align="top-center"/>
 </element>
-<element name="R44" library="SparkFun-Resistors" package="0402-TIGHT" value="10.2Ω" x="59.3217" y="39.8145" smashed="yes">
+<element name="R44" library="SparkFun-Resistors" package="0402-TIGHT" value="10Ω" x="59.3217" y="39.8145" smashed="yes">
 <attribute name="NAME" x="59.3217" y="40.3765" size="0.6096" layer="25" font="vector" ratio="20" align="bottom-center"/>
+<attribute name="PROD_ID" value="RES-16072" x="59.3217" y="39.8145" size="1.778" layer="27" font="vector" ratio="15" display="off"/>
 <attribute name="VALUE" x="61.401959375" y="40.1542" size="0.6096" layer="27" font="vector" ratio="20" align="top-center"/>
 </element>
-<element name="R45" library="SparkFun-Resistors" package="0402-TIGHT" value="10.2Ω" x="58.7984625" y="38.89501875" smashed="yes">
+<element name="R45" library="SparkFun-Resistors" package="0402-TIGHT" value="10Ω" x="58.7984625" y="38.89501875" smashed="yes">
 <attribute name="NAME" x="58.7984625" y="39.45701875" size="0.6096" layer="25" font="vector" ratio="20" align="bottom-center"/>
+<attribute name="PROD_ID" value="RES-16072" x="58.7984625" y="38.89501875" size="1.778" layer="27" font="vector" ratio="15" display="off"/>
 <attribute name="VALUE" x="60.8177625" y="39.1661375" size="0.6096" layer="27" font="vector" ratio="20" align="top-center"/>
 </element>
-<element name="R46" library="SparkFun-Resistors" package="0402-TIGHT" value="5.1Ω" x="61.0108" y="42.4459375" smashed="yes" rot="R180">
+<element name="R46" library="SparkFun-Resistors" package="0402-TIGHT" value="4.7Ω" x="61.0108" y="42.4459375" smashed="yes" rot="R180">
 <attribute name="NAME" x="61.0108" y="41.8839375" size="0.6096" layer="25" font="vector" ratio="20" rot="R180" align="bottom-center"/>
+<attribute name="PROD_ID" value="RES-16312" x="61.0108" y="42.4459375" size="1.778" layer="27" font="vector" ratio="15" rot="R180" display="off"/>
 <attribute name="VALUE" x="62.97168125" y="42.1697375" size="0.6096" layer="27" font="vector" ratio="20" rot="R180" align="top-center"/>
 </element>
-<element name="R47" library="SparkFun-Resistors" package="0402-TIGHT" value="5.1Ω" x="57.058559375" y="42.420540625" smashed="yes" rot="R180">
+<element name="R47" library="SparkFun-Resistors" package="0402-TIGHT" value="4.7Ω" x="57.058559375" y="42.420540625" smashed="yes" rot="R180">
 <attribute name="NAME" x="57.058559375" y="41.858540625" size="0.6096" layer="25" font="vector" ratio="20" rot="R180" align="bottom-center"/>
+<attribute name="PROD_ID" value="RES-16312" x="57.058559375" y="42.420540625" size="1.778" layer="27" font="vector" ratio="15" rot="R180" display="off"/>
 <attribute name="VALUE" x="55.1332375" y="42.1672" size="0.6096" layer="27" font="vector" ratio="20" rot="R180" align="top-center"/>
 </element>
@@
 <attribute name="VALUE" x="105.59038125" y="63.0764" size="0.6096" layer="27" font="vector" ratio="20" rot="R90" align="top-center"/>
 </element>
-<element name="R69" library="SparkFun-Resistors" package="0402-TIGHT" value="10.2Ω" x="97.8281" y="39.8145" smashed="yes">
+<element name="R69" library="SparkFun-Resistors" package="0402-TIGHT" value="10Ω" x="97.8281" y="39.8145" smashed="yes">
 <attribute name="NAME" x="97.8281" y="40.3765" size="0.6096" layer="25" font="vector" ratio="20" align="bottom-center"/>
+<attribute name="PROD_ID" value="RES-16072" x="97.8281" y="39.8145" size="1.778" layer="27" font="vector" ratio="15" display="off"/>
 <attribute name="VALUE" x="99.908359375" y="40.1542" size="0.6096" layer="27" font="vector" ratio="20" align="top-center"/>
 </element>
-<element name="R70" library="SparkFun-Resistors" package="0402-TIGHT" value="10.2Ω" x="97.3048625" y="38.89501875" smashed="yes">
+<element name="R70" library="SparkFun-Resistors" package="0402-TIGHT" value="10Ω" x="97.3048625" y="38.89501875" smashed="yes">
 <attribute name="NAME" x="97.3048625" y="39.45701875" size="0.6096" layer="25" font="vector" ratio="20" align="bottom-center"/>
+<attribute name="PROD_ID" value="RES-16072" x="97.3048625" y="38.89501875" size="1.778" layer="27" font="vector" ratio="15" display="off"/>
 <attribute name="VALUE" x="99.3241625" y="39.1661375" size="0.6096" layer="27" font="vector" ratio="20" align="top-center"/>
 </element>
-<element name="R71" library="SparkFun-Resistors" package="0402-TIGHT" value="5.1Ω" x="99.5172" y="42.4459375" smashed="yes" rot="R180">
+<element name="R71" library="SparkFun-Resistors" package="0402-TIGHT" value="4.7Ω" x="99.5172" y="42.4459375" smashed="yes" rot="R180">
 <attribute name="NAME" x="99.5172" y="41.8839375" size="0.6096" layer="25" font="vector" ratio="20" rot="R180" align="bottom-center"/>
+<attribute name="PROD_ID" value="RES-16312" x="99.5172" y="42.4459375" size="1.778" layer="27" font="vector" ratio="15" rot="R180" display="off"/>
 <attribute name="VALUE" x="101.47808125" y="42.1697375" size="0.6096" layer="27" font="vector" ratio="20" rot="R180" align="top-center"/>
 </element>
-<element name="R72" library="SparkFun-Resistors" package="0402-TIGHT" value="5.1Ω" x="95.564959375" y="42.420540625" smashed="yes" rot="R180">
+<element name="R72" library="SparkFun-Resistors" package="0402-TIGHT" value="4.7Ω" x="95.564959375" y="42.420540625" smashed="yes" rot="R180">
 <attribute name="NAME" x="95.564959375" y="41.858540625" size="0.6096" layer="25" font="vector" ratio="20" rot="R180" align="bottom-center"/>
+<attribute name="PROD_ID" value="RES-16312" x="95.564959375" y="42.420540625" size="1.778" layer="27" font="vector" ratio="15" rot="R180" display="off"/>
 <attribute name="VALUE" x="93.6396375" y="42.1672" size="0.6096" layer="27" font="vector" ratio="20" rot="R180" align="top-center"/>
 </element>
