File: Hardware/Production/SparkFun_MicroMod_Function_ADIN1110-Panel_v11.brd (EAGLE design)
At the start: 127.2 x 157.9 mm, 720 parts, among them J1 IP20(RJ50), J10 IP20(RJ50), J11 MICROMOD_FUNCTION_STANDARD, J12 IP20(RJ50), J2 MICROMOD_FUNCTION_STANDARD, J3 MICROMOD_FUNCTION_STANDARD, J4 IP20(RJ50), J5 MICROMOD_FUNCTION_STANDARD, J6 IP20(RJ50), J7 MICROMOD_FUNCTION_STANDARD, J8 IP20(RJ50), J9 MICROMOD_FUNCTION_STANDARD, Q1 220mA/50V/3.5Ω, Q10 220mA/50V/3.5Ω, Q11 20V/4.2A/52mΩ/1.4W, Q12 220mA/50V/3.5Ω, Q2 20V/4.2A/52mΩ/1.4W, Q3 20V/4.2A/52mΩ/1.4W, Q4 220mA/50V/3.5Ω, Q5 20V/4.2A/52mΩ/1.4W, Q6 220mA/50V/3.5Ω, Q7 20V/4.2A/52mΩ/1.4W, Q8 220mA/50V/3.5Ω, Q9 20V/4.2A/52mΩ/1.4W, T1 WE-STST, T2 WE-STST, T3 WE-STST, T4 WE-STST, T5 WE-STST, T6 WE-STST, U1 ADIN1110, U10 3.3V, U11 ADIN1110, U12 WE-TVS, U13 EEPROM, U14 3.3V, U15 ADIN1110, U16 WE-TVS, U17 EEPROM, U18 3.3V, U19 ADIN1110, U2 EEPROM, U20 WE-TVS, U21 EEPROM, U22 3.3V, U23 ADIN1110, U24 WE-TVS, U3 3.3V, U4 WE-TVS, U5 EEPROM, U6 3.3V, U7 ADIN1110, U8 WE-TVS, U9 EEPROM, Y1 25MHz, Y2 25MHz, Y3 25MHz, Y4 25MHz, Y5 25MHz, Y6 25MHz

Commit message: R27 changed to 4.7K
-updated prod_id and values on boat single and panel files.
Parts:
- R114, R143, R172, R27, R56, R85: value 10k -> 4.7K
Changed lines of the file:
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@@
 <layer number="19" name="Unrouted" color="6" fill="1" visible="yes" active="yes"/>
 <layer number="20" name="Dimension" color="24" fill="1" visible="yes" active="yes"/>
-<layer number="21" name="tPlace" color="7" fill="1" visible="yes" active="yes"/>
-<layer number="22" name="bPlace" color="7" fill="1" visible="yes" active="yes"/>
+<layer number="21" name="tPlace" color="16" fill="1" visible="yes" active="yes"/>
+<layer number="22" name="bPlace" color="14" fill="1" visible="yes" active="yes"/>
 <layer number="23" name="tOrigins" color="15" fill="1" visible="yes" active="yes"/>
 <layer number="24" name="bOrigins" color="15" fill="1" visible="yes" active="yes"/>
@@
 <layer number="49" name="Reference" color="7" fill="1" visible="yes" active="yes"/>
 <layer number="50" name="dxf" color="7" fill="1" visible="yes" active="yes"/>
-<layer number="51" name="tDocu" color="7" fill="1" visible="yes" active="yes"/>
+<layer number="51" name="tDocu" color="6" fill="1" visible="yes" active="yes"/>
 <layer number="52" name="bDocu" color="7" fill="1" visible="yes" active="yes"/>
 <layer number="53" name="tGND_GNDA" color="7" fill="9" visible="no" active="no"/>
@@
 <attribute name="VALUE" x="9.6774" y="10.414" size="0.6096" layer="27" font="vector" ratio="20" rot="R270" align="top-center"/>
 </element>
-<element name="R27" library="SparkFun-Resistors" package="0603" value="10k" x="26.416" y="45.72" smashed="yes" rot="R90">
+<element name="R27" library="SparkFun-Resistors" package="0603" value="4.7K" x="26.416" y="45.72" smashed="yes" rot="R90">
 <attribute name="NAME" x="25.654" y="45.72" size="0.6096" layer="25" font="vector" ratio="20" rot="R90" align="bottom-center"/>
-<attribute name="PROD_ID" value="RES-00824" x="26.416" y="45.72" size="1.778" layer="27" font="vector" ratio="15" rot="R90" display="off"/>
+<attribute name="PROD_ID" value="RES-07857" x="26.416" y="45.72" size="1.778" layer="27" font="vector" ratio="15" rot="R90" display="off"/>
 <attribute name="VALUE" x="27.178" y="45.72" size="0.6096" layer="27" font="vector" ratio="20" rot="R90" align="top-center"/>
 </element>
@@
 <attribute name="VALUE" x="47.6758" y="10.414" size="0.6096" layer="27" font="vector" ratio="20" rot="R270" align="top-center"/>
 </element>
-<element name="R56" library="SparkFun-Resistors" package="0603" value="10k" x="64.4144" y="45.72" smashed="yes" rot="R90">
+<element name="R56" library="SparkFun-Resistors" package="0603" value="4.7K" x="64.4144" y="45.72" smashed="yes" rot="R90">
 <attribute name="NAME" x="63.6524" y="45.72" size="0.6096" layer="25" font="vector" ratio="20" rot="R90" align="bottom-center"/>
-<attribute name="PROD_ID" value="RES-00824" x="64.4144" y="45.72" size="1.778" layer="27" font="vector" ratio="15" rot="R90" display="off"/>
+<attribute name="PROD_ID" value="RES-07857" x="64.4144" y="45.72" size="1.778" layer="27" font="vector" ratio="15" rot="R90" display="off"/>
 <attribute name="VALUE" x="65.1764" y="45.72" size="0.6096" layer="27" font="vector" ratio="20" rot="R90" align="top-center"/>
 </element>
@@
 <attribute name="VALUE" x="85.6742" y="10.414" size="0.6096" layer="27" font="vector" ratio="20" rot="R270" align="top-center"/>
 </element>
-<element name="R85" library="SparkFun-Resistors" package="0603" value="10k" x="102.4128" y="45.72" smashed="yes" rot="R90">
+<element name="R85" library="SparkFun-Resistors" package="0603" value="4.7K" x="102.4128" y="45.72" smashed="yes" rot="R90">
 <attribute name="NAME" x="101.6508" y="45.72" size="0.6096" layer="25" font="vector" ratio="20" rot="R90" align="bottom-center"/>
-<attribute name="PROD_ID" value="RES-00824" x="102.4128" y="45.72" size="1.778" layer="27" font="vector" ratio="15" rot="R90" display="off"/>
+<attribute name="PROD_ID" value="RES-07857" x="102.4128" y="45.72" size="1.778" layer="27" font="vector" ratio="15" rot="R90" display="off"/>
 <attribute name="VALUE" x="103.1748" y="45.72" size="0.6096" layer="27" font="vector" ratio="20" rot="R90" align="top-center"/>
 </element>
@@
 <attribute name="VALUE" x="27.813" y="128.475740625" size="0.6096" layer="27" font="vector" ratio="20" rot="R90" align="top-center"/>
 </element>
-<element name="R114" library="SparkFun-Resistors" package="0603" value="10k" x="11.0744" y="93.169740625" smashed="yes" rot="R270">
+<element name="R114" library="SparkFun-Resistors" package="0603" value="4.7K" x="11.0744" y="93.169740625" smashed="yes" rot="R270">
 <attribute name="NAME" x="11.8364" y="93.169740625" size="0.6096" layer="25" font="vector" ratio="20" rot="R270" align="bottom-center"/>
-<attribute name="PROD_ID" value="RES-00824" x="11.0744" y="93.169740625" size="1.778" layer="27" font="vector" ratio="15" rot="R270" display="off"/>
+<attribute name="PROD_ID" value="RES-07857" x="11.0744" y="93.169740625" size="1.778" layer="27" font="vector" ratio="15" rot="R270" display="off"/>
 <attribute name="VALUE" x="10.3124" y="93.169740625" size="0.6096" layer="27" font="vector" ratio="20" rot="R270" align="top-center"/>
 </element>
@@
 <attribute name="VALUE" x="65.8114" y="128.475740625" size="0.6096" layer="27" font="vector" ratio="20" rot="R90" align="top-center"/>
 </element>
-<element name="R143" library="SparkFun-Resistors" package="0603" value="10k" x="49.0728" y="93.169740625" smashed="yes" rot="R270">
+<element name="R143" library="SparkFun-Resistors" package="0603" value="4.7K" x="49.0728" y="93.169740625" smashed="yes" rot="R270">
 <attribute name="NAME" x="49.8348" y="93.169740625" size="0.6096" layer="25" font="vector" ratio="20" rot="R270" align="bottom-center"/>
-<attribute name="PROD_ID" value="RES-00824" x="49.0728" y="93.169740625" size="1.778" layer="27" font="vector" ratio="15" rot="R270" display="off"/>
+<attribute name="PROD_ID" value="RES-07857" x="49.0728" y="93.169740625" size="1.778" layer="27" font="vector" ratio="15" rot="R270" display="off"/>
 <attribute name="VALUE" x="48.3108" y="93.169740625" size="0.6096" layer="27" font="vector" ratio="20" rot="R270" align="top-center"/>
 </element>
@@
 <attribute name="VALUE" x="103.8098" y="128.475740625" size="0.6096" layer="27" font="vector" ratio="20" rot="R90" align="top-center"/>
 </element>
-<element name="R172" library="SparkFun-Resistors" package="0603" value="10k" x="87.0712" y="93.169740625" smashed="yes" rot="R270">
+<element name="R172" library="SparkFun-Resistors" package="0603" value="4.7K" x="87.0712" y="93.169740625" smashed="yes" rot="R270">
 <attribute name="NAME" x="87.8332" y="93.169740625" size="0.6096" layer="25" font="vector" ratio="20" rot="R270" align="bottom-center"/>
-<attribute name="PROD_ID" value="RES-00824" x="87.0712" y="93.169740625" size="1.778" layer="27" font="vector" ratio="15" rot="R270" display="off"/>
+<attribute name="PROD_ID" value="RES-07857" x="87.0712" y="93.169740625" size="1.778" layer="27" font="vector" ratio="15" rot="R270" display="off"/>
 <attribute name="VALUE" x="86.3092" y="93.169740625" size="0.6096" layer="27" font="vector" ratio="20" rot="R270" align="top-center"/>
 </element>
