File: Hardware/Production/SparkFun_MicroMod_Function_ADIN1110-Panel_v12.brd (EAGLE design)
At the start: 127.2 x 157.9 mm, 720 parts, among them J1 IP20(RJ50), J10 IP20(RJ50), J11 MICROMOD_FUNCTION_STANDARD, J12 IP20(RJ50), J2 MICROMOD_FUNCTION_STANDARD, J3 MICROMOD_FUNCTION_STANDARD, J4 IP20(RJ50), J5 MICROMOD_FUNCTION_STANDARD, J6 IP20(RJ50), J7 MICROMOD_FUNCTION_STANDARD, J8 IP20(RJ50), J9 MICROMOD_FUNCTION_STANDARD, Q1 220mA/50V/3.5Ω, Q10 220mA/50V/3.5Ω, Q11 20V/4.2A/52mΩ/1.4W, Q12 220mA/50V/3.5Ω, Q2 20V/4.2A/52mΩ/1.4W, Q3 20V/4.2A/52mΩ/1.4W, Q4 220mA/50V/3.5Ω, Q5 20V/4.2A/52mΩ/1.4W, Q6 220mA/50V/3.5Ω, Q7 20V/4.2A/52mΩ/1.4W, Q8 220mA/50V/3.5Ω, Q9 20V/4.2A/52mΩ/1.4W, T1 WE-STST, T2 WE-STST, T3 WE-STST, T4 WE-STST, T5 WE-STST, T6 WE-STST, U1 ADIN1110, U10 3.3V, U11 ADIN1110, U12 WE-TVS, U13 EEPROM, U14 3.3V, U15 ADIN1110, U16 WE-TVS, U17 EEPROM, U18 3.3V, U19 ADIN1110, U2 EEPROM, U20 WE-TVS, U21 EEPROM, U22 3.3V, U23 ADIN1110, U24 WE-TVS, U3 3.3V, U4 WE-TVS, U5 EEPROM, U6 3.3V, U7 ADIN1110, U8 WE-TVS, U9 EEPROM, Y1 25MHz, Y2 25MHz, Y3 25MHz, Y4 25MHz, Y5 25MHz, Y6 25MHz

Commit message: Removed v11 panel and added v12 panel
Parts:
- added U$169, U$205: (no value), output:##SWPD_EN##4
- added U$170, U$171, U$206, U$207: (no value), output:SINGLE_PAIR_ETHERNET0
- added U$172, U$208: (no value), temp_logos:ANALOG_DEVICE_LOGO_9MM
- added U$173, U$209: (no value), temp_logos:HARTING_LOGO_9MM
- added U$174, U$210: (no value), temp_logos:WURTH_LOGO_9MM
- added U$175, U$211: (no value), temp_logos:DIGIKEY_LOGO
- added U$176, U$212: (no value), SparkFun-Aesthetics:SFE_LOGO_NAME_FLAME_.1
- added U$177, U$213: DIGIKEY_LOGO, temp_logos:DIGIKEY_LOGO
- added U$178, U$214: ANALOG_DEVICES_LOGO, temp_logos:ANALOG_DEVICE_LOGO_9MM
- added U$179, U$215: HARTING_LOGO, temp_logos:HARTING_LOGO_9MM
- added U$180, U$216: WURTH_LOGO, temp_logos:WURTH_LOGO_9MM
- added U$181, U$182: (no value), SparkFun-MicroMod:MICROMOD_LOGO_.35
- added U$183: (no value), output:#MEAS#3
- added U$184: (no value), output:PWR0
- added U$185, U$193: (no value), output:FUNCTION0
- added U$186, U$192: (no value), output:ADIN11100
- added U$187: (no value), output:#RESET#0
- added U$188: (no value), output:SHLD11
- added U$189: (no value), output:#SPI_CFG1#0
- added U$190: (no value), output:#MS_SEL#2
- added U$191: (no value), output:#SPI_CFG0#0
- added U$194: (no value), output:LED_03
- added U$195: (no value), output:LED_14
- added U$196: (no value), output:LINK_ST15
- added U$197: (no value), output:#GND#16
- added U$198: (no value), output:#CAP#17
- added U$199: (no value), output:#EWP#18
- added U$200: (no value), output:#PWR#19
- added U$201: (no value), output:#LED0#20
- added U$202: (no value), output:#LED1#21
- added U$203: (no value), ADIN1110:#LINKST#2
- added U$204: (no value), output:##TX2P4_EN##4
- CIPO, CIPO1, CIPO2, CIPO3, CIPO4, CIPO5, COPI, COPI1, COPI2, COPI3, COPI4, COPI5, CS, CS1, CS2, CS3, CS4, CS5, INT, INT1, INT2, INT3, INT4, INT5, SPI, SPI1, SPI2, SPI3, SPI4, SPI5: value (none) -> TEST-POINTTP_15TH_THRU
- LOGO1, LOGO10, LOGO12, LOGO4, LOGO6, LOGO8: value SFE_LOGO_NAME_FLAME.2_INCH -> SFE_LOGO_NAME_FLAME.1_INCH; device SparkFun-Aesthetics:SFE_LOGO_NAME_FLAME_.2 -> SparkFun-Aesthetics:SFE_LOGO_NAME_FLAME_.1
- R114, R143, R172, R27, R56, R85: value 4.7K -> 4.7k
- U$100: device output:LED_14 -> temp_logos:ANALOG_DEVICE_LOGO_9MM
- U$101: device output:LINK_ST15 -> temp_logos:HARTING_LOGO_9MM
- U$102: device output:#GND#16 -> temp_logos:WURTH_LOGO_9MM
- U$103: device output:#CAP#17 -> temp_logos:DIGIKEY_LOGO
- U$104: device output:#EWP#18 -> SparkFun-Aesthetics:SFE_LOGO_NAME_FLAME_.1
- U$105: value (none) -> DIGIKEY_LOGO; device output:#PWR#19 -> temp_logos:DIGIKEY_LOGO
- U$106: value (none) -> ANALOG_DEVICES_LOGO; device output:#LED0#20 -> temp_logos:ANALOG_DEVICE_LOGO_9MM
- U$107: value (none) -> HARTING_LOGO; device output:#LED1#21 -> temp_logos:HARTING_LOGO_9MM
- U$108: value (none) -> WURTH_LOGO; device ADIN1110:#LINKST#2 -> temp_logos:WURTH_LOGO_9MM
- U$109: device output:##TX2P4_EN##4 -> SparkFun-MicroMod:MICROMOD_LOGO_.35
- U$110: device output:##SWPD_EN##4 -> SparkFun-MicroMod:MICROMOD_LOGO_.35
- U$111: device output:SINGLE_PAIR_ETHERNET0 -> output:#MEAS#3
- U$112: device output:SINGLE_PAIR_ETHERNET0 -> output:PWR0
- U$113, U$85: device SparkFun-MicroMod:MICROMOD_LOGO_.35 -> output:FUNCTION0
- U$114: device SparkFun-MicroMod:MICROMOD_LOGO_.35 -> output:ADIN11100
- U$115: device output:#MEAS#3 -> output:#RESET#0
- U$116: device output:PWR0 -> output:SHLD11
- U$117: device output:FUNCTION0 -> output:#SPI_CFG1#0
- U$118: device output:ADIN11100 -> output:#MS_SEL#2
- U$119: device SparkFun-Aesthetics:SFE_LOGO_FLAME_.1 -> output:#SPI_CFG0#0
- U$120: device output:#RESET#0 -> output:ADIN11100
- U$121, U$149: device output:SHLD11 -> output:FUNCTION0
- U$122: device output:#SPI_CFG1#0 -> output:LED_03
- U$123: device output:#MS_SEL#2 -> output:LED_14
- U$124: device output:#SPI_CFG0#0 -> output:LINK_ST15
- U$125: device output:ADIN11100 -> output:#GND#16
- U$126: device output:FUNCTION0 -> output:#CAP#17
- U$127: device output:LED_03 -> output:#EWP#18
- U$128: device output:LED_14 -> output:#PWR#19
- U$129: device output:LINK_ST15 -> output:#LED0#20
- U$130: device output:#GND#16 -> output:#LED1#21
- U$131: device output:#CAP#17 -> ADIN1110:#LINKST#2
- U$132: device output:#EWP#18 -> output:##TX2P4_EN##4
- U$133: device output:#PWR#19 -> output:##SWPD_EN##4
- U$134: device output:#LED0#20 -> output:SINGLE_PAIR_ETHERNET0
- U$135: device output:#LED1#21 -> output:SINGLE_PAIR_ETHERNET0
- U$136: device ADIN1110:#LINKST#2 -> temp_logos:ANALOG_DEVICE_LOGO_9MM
- U$137: device output:##TX2P4_EN##4 -> temp_logos:HARTING_LOGO_9MM
- U$138: device output:##SWPD_EN##4 -> temp_logos:WURTH_LOGO_9MM
- U$139: device output:SINGLE_PAIR_ETHERNET0 -> temp_logos:DIGIKEY_LOGO
- U$140: device output:SINGLE_PAIR_ETHERNET0 -> SparkFun-Aesthetics:SFE_LOGO_NAME_FLAME_.1
- U$141: value (none) -> DIGIKEY_LOGO; device SparkFun-MicroMod:MICROMOD_LOGO_.35 -> temp_logos:DIGIKEY_LOGO
- U$142: value (none) -> ANALOG_DEVICES_LOGO; device SparkFun-MicroMod:MICROMOD_LOGO_.35 -> temp_logos:ANALOG_DEVICE_LOGO_9MM
- U$143: value (none) -> HARTING_LOGO; device output:#MEAS#3 -> temp_logos:HARTING_LOGO_9MM
- U$144: value (none) -> WURTH_LOGO; device output:PWR0 -> temp_logos:WURTH_LOGO_9MM
- U$145: device output:FUNCTION0 -> SparkFun-MicroMod:MICROMOD_LOGO_.35
- U$146: device output:ADIN11100 -> SparkFun-MicroMod:MICROMOD_LOGO_.35
- U$147: device SparkFun-Aesthetics:SFE_LOGO_FLAME_.1 -> output:#MEAS#3
- U$148: device output:#RESET#0 -> output:PWR0
- U$150: device output:#SPI_CFG1#0 -> output:ADIN11100
- U$151: device output:#MS_SEL#2 -> output:#RESET#0
- U$152: device output:#SPI_CFG0#0 -> output:SHLD11
- U$153: device output:ADIN11100 -> output:#SPI_CFG1#0
- U$154: device output:FUNCTION0 -> output:#MS_SEL#2
- U$155: device output:LED_03 -> output:#SPI_CFG0#0
- U$156: device output:LED_14 -> output:ADIN11100
- U$157: device output:LINK_ST15 -> output:FUNCTION0
- U$158: device output:#GND#16 -> output:LED_03
- U$159: device output:#CAP#17 -> output:LED_14
- U$160: device output:#EWP#18 -> output:LINK_ST15
- U$161: device output:#PWR#19 -> output:#GND#16
- U$162: device output:#LED0#20 -> output:#CAP#17
- U$163: device output:#LED1#21 -> output:#EWP#18
- U$164: device ADIN1110:#LINKST#2 -> output:#PWR#19
- U$165: device output:##TX2P4_EN##4 -> output:#LED0#20
- U$166: device output:##SWPD_EN##4 -> output:#LED1#21
- U$167: device output:SINGLE_PAIR_ETHERNET0 -> ADIN1110:#LINKST#2
- U$168: device output:SINGLE_PAIR_ETHERNET0 -> output:##TX2P4_EN##4
- U$19: value (none) -> WURTH_LOGO; device output:#MEAS#3 -> temp_logos:WURTH_LOGO_9MM
- U$2: value (none) -> HARTING_LOGO; device SparkFun-MicroMod:MICROMOD_LOGO_.35 -> temp_logos:HARTING_LOGO_9MM
- U$20: device output:PWR0 -> temp_logos:ANALOG_DEVICE_LOGO_9MM
- U$30: device output:FUNCTION0 -> temp_logos:HARTING_LOGO_9MM
- U$32: device output:ADIN11100 -> temp_logos:WURTH_LOGO_9MM
- U$33: value (none) -> ANALOG_DEVICES_LOGO; device SparkFun-Aesthetics:SFE_LOGO_FLAME_.1 -> temp_logos:ANALOG_DEVICE_LOGO_9MM
- U$34: device output:#RESET#0 -> temp_logos:DIGIKEY_LOGO
- U$35: device output:SHLD11 -> SparkFun-Aesthetics:SFE_LOGO_NAME_FLAME_.1
- U$36: device output:#SPI_CFG1#0 -> SparkFun-MicroMod:MICROMOD_LOGO_.35
- U$38: device output:#MS_SEL#2 -> output:#MEAS#3
- U$39: device output:#SPI_CFG0#0 -> output:PWR0
- U$40: device output:ADIN11100 -> output:FUNCTION0
- U$41: device output:FUNCTION0 -> output:ADIN11100
- U$42: device output:LED_03 -> output:#RESET#0
- U$43: device output:LED_14 -> output:SHLD11
- U$44: device output:LINK_ST15 -> output:#SPI_CFG1#0
- U$45: device output:#GND#16 -> output:#MS_SEL#2
- U$46: device output:#CAP#17 -> output:#SPI_CFG0#0
- U$47: device output:#EWP#18 -> output:ADIN11100
- U$48, U$77: device output:#PWR#19 -> output:FUNCTION0
- U$49: device output:#LED0#20 -> output:LED_03
- U$5: value (none) -> DIGIKEY_LOGO; device SparkFun-Aesthetics:SFE_LOGO_FLAME_.1 -> temp_logos:DIGIKEY_LOGO
- U$50: device output:#LED1#21 -> output:LED_14
- U$51: device ADIN1110:#LINKST#2 -> output:LINK_ST15
- U$52: device output:##TX2P4_EN##4 -> output:#GND#16
- U$53: device output:##SWPD_EN##4 -> output:#CAP#17
- U$54: device output:SINGLE_PAIR_ETHERNET0 -> output:#EWP#18
- U$55: device output:SINGLE_PAIR_ETHERNET0 -> output:#PWR#19
- U$56: device SparkFun-MicroMod:MICROMOD_LOGO_.35 -> output:#LED0#20
- U$57: device SparkFun-MicroMod:MICROMOD_LOGO_.35 -> output:#LED1#21
- U$58: device output:#MEAS#3 -> ADIN1110:#LINKST#2
- U$59: device output:PWR0 -> output:##TX2P4_EN##4
- U$60: device output:FUNCTION0 -> output:##SWPD_EN##4
- U$61: device output:ADIN11100 -> output:SINGLE_PAIR_ETHERNET0
- U$62: device SparkFun-Aesthetics:SFE_LOGO_FLAME_.1 -> output:SINGLE_PAIR_ETHERNET0
- U$64: device output:#RESET#0 -> temp_logos:ANALOG_DEVICE_LOGO_9MM
- U$65: device output:SHLD11 -> temp_logos:HARTING_LOGO_9MM
- U$66: device output:#SPI_CFG1#0 -> temp_logos:WURTH_LOGO_9MM
- U$67: device output:#MS_SEL#2 -> temp_logos:DIGIKEY_LOGO
- U$68: device output:#SPI_CFG0#0 -> SparkFun-Aesthetics:SFE_LOGO_NAME_FLAME_.1
- U$69: value (none) -> DIGIKEY_LOGO; device output:ADIN11100 -> temp_logos:DIGIKEY_LOGO
- U$70: value (none) -> ANALOG_DEVICES_LOGO; device output:FUNCTION0 -> temp_logos:ANALOG_DEVICE_LOGO_9MM
- U$71: value (none) -> HARTING_LOGO; device output:LED_03 -> temp_logos:HARTING_LOGO_9MM
- U$72: value (none) -> WURTH_LOGO; device output:LED_14 -> temp_logos:WURTH_LOGO_9MM
- U$73: device output:LINK_ST15 -> SparkFun-MicroMod:MICROMOD_LOGO_.35
- U$74: device output:#GND#16 -> SparkFun-MicroMod:MICROMOD_LOGO_.35
- U$75: device output:#CAP#17 -> output:#MEAS#3
- U$76: device output:#EWP#18 -> output:PWR0
- U$78: device output:#LED0#20 -> output:ADIN11100
- U$79: device output:#LED1#21 -> output:#RESET#0
- U$80: device ADIN1110:#LINKST#2 -> output:SHLD11
- U$81: device output:##TX2P4_EN##4 -> output:#SPI_CFG1#0
- U$82: device output:##SWPD_EN##4 -> output:#MS_SEL#2
- U$83: device output:SINGLE_PAIR_ETHERNET0 -> output:#SPI_CFG0#0
- U$84: device output:SINGLE_PAIR_ETHERNET0 -> output:ADIN11100
- U$86: device SparkFun-MicroMod:MICROMOD_LOGO_.35 -> output:LED_03
- U$87: device output:#MEAS#3 -> output:LED_14
- U$88: device output:PWR0 -> output:LINK_ST15
- U$89: device output:FUNCTION0 -> output:#GND#16
- U$90: device output:ADIN11100 -> output:#CAP#17
- U$91: device SparkFun-Aesthetics:SFE_LOGO_FLAME_.1 -> output:#EWP#18
- U$92: device output:#RESET#0 -> output:#PWR#19
- U$93: device output:SHLD11 -> output:#LED0#20
- U$94: device output:#SPI_CFG1#0 -> output:#LED1#21
- U$95: device output:#MS_SEL#2 -> ADIN1110:#LINKST#2
- U$96: device output:#SPI_CFG0#0 -> output:##TX2P4_EN##4
- U$97: device output:ADIN11100 -> output:##SWPD_EN##4
- U$98: device output:FUNCTION0 -> output:SINGLE_PAIR_ETHERNET0
- U$99: device output:LED_03 -> output:SINGLE_PAIR_ETHERNET0
- moved U$106 142.9 mm to (107.6, 11.4), flipped to the top, turned to 0 degrees
- moved U$107 132.1 mm to (105.3, 19.8), flipped to the top, turned to 0 degrees
- moved U$91 126.4 mm to (97.2, 14.2), flipped to the bottom, turned to 0 degrees
- moved U$96 126.0 mm to (88.4, 25.4), turned to 0 degrees
- moved U$108 121.6 mm to (88.3, 19.9), flipped to the top, turned to 0 degrees
- moved U$92 121.3 mm to (109.4, 26.7), flipped to the bottom, turned to 0 degrees
- moved U$94 120.7 mm to (109.5, 34.3), turned to 0 degrees
- moved U$95 120.7 mm to (109.9, 31.8), turned to 0 degrees
- moved U$142 113.9 mm to (5.87, 127.5), flipped to the top
- moved U$105 106.0 mm to (85.3, 43.9), flipped to the top, turned to 0 degrees
- moved U$97 104.7 mm to (88.1, 22.9), turned to 0 degrees
- moved U$101 104.5 mm to (86.8, 9.27), flipped to the bottom, turned to 0 degrees
- moved U$143 104.4 mm to (8.15, 119.1), flipped to the top, turned to 180 degrees
- moved U$102 104.3 mm to (101.5, 9.14), turned to 0 degrees
- moved U$88 103.4 mm to (103.7, 58.9), turned to 90 degrees
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Connections:
- net GND: now also J2.2, J2.8
- net GND1: now also J3.2, J3.8
- net GND2: now also J5.2, J5.8
- net GND3: now also J7.2, J7.8
- net GND4: now also J9.2, J9.8
- net GND5: now also J11.2, J11.8
Other:
- board size 127.2 x 157.9 mm -> 127.2 x 160.5 mm
- board text added: "v12"
- board text removed: "v11"
