File: Hardware/SparkFun_MicroMod_Function_ADIN1110.sch (EAGLE design)
At the start: 83 parts, among them J1 T1_INDUSTRIAL, J2 MICROMOD_FUNCTION_STANDARD, Q1 220mA/50V/3.5Ω, Q2 20V/4.2A/52mΩ/1.4W, T1 WE-STST, U1 ADIN1110, U2 EEPROM, U3 3.3V, U4 WE-TVS, Y1 25MHz

Commit message: Wurth Electronik caps
Parts:
- C10, C13, C15, C16, C18: device SparkFun-Capacitors:0.1UF-0402T-16V-10% -> SparkFun-Capacitors:0.1UF-0402T-16V-10%-X7R-WE
- C12, C14, C17: device SparkFun-Capacitors:10NF-0402T-25V-10% -> SparkFun-Capacitors:10NF-0402T-25V-10%-X7R-WE
- C21: value 0.1uF/50V -> 0.1uF
- C22: value 0.1uF/100V -> 0.1uF
- C3, C4: device SparkFun-Capacitors:0.1UF-0603-25V-(+80/-20%) -> SparkFun-Capacitors:0.1UF-0603-25V-10%-X7R-WE
- C5, C6: device SparkFun-Capacitors:10PF-0603-50V-5% -> SparkFun-Capacitors:10PF-0603-50V-5%-C0G-WE
- C7: device SparkFun-Capacitors:3.3NF-0603-100V-10% -> SparkFun-Capacitors:3.3NF-0603-100V-10%-WE
- C8: device SparkFun-Capacitors:1.0UF-0603-16V-10% -> SparkFun-Capacitors:1.0UF-0603-16V-10%-X7R-WE
- C9: device SparkFun-Capacitors:1.0UF-0603-16V-10%-X7R -> SparkFun-Capacitors:1.0UF-0603-16V-10%-X7R-WE

Commit message: LEDs and Xtal swapped out for Wurth Electronic Parts
Also bumped version to v10, because the WE xtal has GND pads, and new package has polarity dot.
Parts:
- LED_0: device SparkFun-LED:LED-GREEN0603 -> SparkFun-LED:LED-GREEN-0603-WE
- LED_1: device SparkFun-LED:LED-YELLOW0603 -> SparkFun-LED:LED-YELLOW-0603-WE
- LINK_ST: device SparkFun-LED:LED-BLUE0603 -> SparkFun-LED:LED-BLUE-0603-WE
- PWR: device SparkFun-LED:LED-RED0603 -> SparkFun-LED:LED-RED-0603-WE
- Y1: device SparkFun-Clocks:CRYSTAL-25MHZ-SMD-2.0X1.6MM -> SparkFun-Clocks:CRYSTAL-25MHZ-WE-SMD-2.0X1.6MM-WE
Connections:
- net GND: now also Y1.GND
Other:
- note added: "v10"
- note removed: "v01"
Changed lines of the file:
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@@
 <part name="GND10" library="SparkFun-PowerSymbols" deviceset="GND" device=""/>
 <part name="LOGO2" library="SparkFun-Aesthetics" deviceset="SPECIAL_INSTRUCTIONS" device="-ORDERING"/>
-<part name="Y1" library="SparkFun-Clocks" deviceset="CRYSTAL-25MHZ" device="-SMD-2.0X1.6MM" value="25MHz"/>
+<part name="Y1" library="SparkFun-Clocks" deviceset="CRYSTAL-25MHZ-WE" device="-SMD-2.0X1.6MM-WE" value="25MHz"/>
 <part name="C5" library="SparkFun-Capacitors" deviceset="10PF" device="-0603-50V-5%-C0G-WE" value="10pF"/>
 <part name="C6" library="SparkFun-Capacitors" deviceset="10PF" device="-0603-50V-5%-C0G-WE" value="10pF"/>
@@
 <part name="LED-PWR" library="SparkFun-Jumpers" deviceset="JUMPER-SMT_2_NC_TRACE" device="_SILK" package3d_urn="urn:adsk.eagle:package:39281/1" value="JUMPER-SMT_2_NC_TRACE_SILK"/>
 <part name="R9" library="SparkFun-Resistors" deviceset="1KOHM" device="-0402T-1/16W-1%" value="1k"/>
-<part name="PWR" library="SparkFun-LED" deviceset="LED-RED" device="0603" value="Red"/>
+<part name="PWR" library="SparkFun-LED" deviceset="LED-RED" device="-0603-WE" value="Red"/>
 <part name="GND33" library="SparkFun-PowerSymbols" deviceset="GND" device=""/>
 <part name="SUPPLY5" library="SparkFun-PowerSymbols" deviceset="3.3V" device=""/>
@@
 <part name="C19" library="SparkFun-Capacitors" deviceset="1.0UF" device="-0402T-16V-10%" value="1.0uF"/>
 <part name="GND45" library="SparkFun-PowerSymbols" deviceset="GND" device=""/>
-<part name="LED_0" library="SparkFun-LED" deviceset="LED-GREEN" device="0603" value="Green"/>
+<part name="LED_0" library="SparkFun-LED" deviceset="LED-GREEN" device="-0603-WE" value="Green"/>
 <part name="R11" library="SparkFun-Resistors" deviceset="1KOHM" device="-0402T-1/16W-1%" value="1k"/>
 <part name="SWPD" library="SparkFun-Jumpers" deviceset="JUMPER-SMT_2_NO" device="_SILK" package3d_urn="urn:adsk.eagle:package:39279/1" value=""/>
@@
 <part name="SUPPLY30" library="SparkFun-PowerSymbols" deviceset="3.3V" device=""/>
 <part name="SUPPLY31" library="SparkFun-PowerSymbols" deviceset="3.3V" device=""/>
-<part name="LED_1" library="SparkFun-LED" deviceset="LED-YELLOW" device="0603" value="Yellow"/>
+<part name="LED_1" library="SparkFun-LED" deviceset="LED-YELLOW" device="-0603-WE" value="Yellow"/>
 <part name="R21" library="SparkFun-Resistors" deviceset="1KOHM" device="-0402T-1/16W-1%" value="1k"/>
 <part name="R19" library="SparkFun-Resistors" deviceset="4.7KOHM" device="-0402T-1/16W-1%" value="4.7k"/>
-<part name="LINK_ST" library="SparkFun-LED" deviceset="LED-BLUE" device="0603" value="Blue"/>
+<part name="LINK_ST" library="SparkFun-LED" deviceset="LED-BLUE" device="-0603-WE" value="Blue"/>
 <part name="GND46" library="SparkFun-PowerSymbols" deviceset="GND" device=""/>
 <part name="GND47" library="SparkFun-PowerSymbols" deviceset="GND" device=""/>
@@
 <part name="R25" library="SparkFun-Resistors" deviceset="4.7KOHM" device="-0402T-1/16W-1%" value="4.7k"/>
 <part name="SUPPLY3" library="SparkFun-PowerSymbols" deviceset="3.3V" device=""/>
+<part name="GND15" library="SparkFun-PowerSymbols" deviceset="GND" device=""/>
 </parts>
 <sheets>
@@
 <text x="30.734" y="126.746" size="2.54" layer="94" font="vector" ratio="12" align="center">MicroMod Function Connector</text>
 <text x="348.996" y="11.684" size="1.778" layer="94" font="vector">Pete Lewis</text>
-<text x="421.894" y="6.096" size="2.54" layer="94" font="vector">v01</text>
+<text x="421.894" y="6.096" size="2.54" layer="94" font="vector">v10</text>
 <text x="45.72" y="271.78" size="2.54" layer="94" font="vector" ratio="12" align="center">ADIN1110 BASE10-T1L ETHERNET MAC-PHY</text>
 <text x="317.754" y="124.206" size="2.54" layer="94" font="vector" ratio="12" align="center">Power Enable</text>
@@
 </instance>
 <instance part="LOGO2" gate="G$1" x="408.94" y="22.86" smashed="yes"/>
-<instance part="Y1" gate="Y1" x="58.42" y="182.88" smashed="yes">
-<attribute name="NAME" x="58.42" y="178.816" size="1.778" layer="95" font="vector" align="bottom-center"/>
+<instance part="Y1" gate="G$1" x="58.42" y="182.88" smashed="yes">
+<attribute name="NAME" x="60.198" y="178.816" size="1.778" layer="95" font="vector" align="bottom-center"/>
 <attribute name="VALUE" x="58.42" y="185.166" size="1.778" layer="96" font="vector" rot="R180" align="top-center"/>
 </instance>
@@
 <attribute name="VALUE" x="134.62" y="73.914" size="1.778" layer="96" font="vector" align="bottom-center"/>
 </instance>
+<instance part="GND15" gate="1" x="58.42" y="167.64" smashed="yes">
+<attribute name="VALUE" x="58.42" y="167.386" size="1.778" layer="96" font="vector" align="top-center"/>
+</instance>
 </instances>
 <busses>
@@
 <wire x1="256.54" y1="160.02" x2="256.54" y2="157.48" width="0.1524" layer="91"/>
 <pinref part="GND14" gate="1" pin="GND"/>
+</segment>
+<segment>
+<pinref part="Y1" gate="G$1" pin="GND"/>
+<pinref part="GND15" gate="1" pin="GND"/>
+<wire x1="58.42" y1="177.8" x2="58.42" y2="170.18" width="0.1524" layer="91"/>
 </segment>
 </net>
@@
 <wire x1="93.98" y1="187.96" x2="50.8" y2="187.96" width="0.1524" layer="91"/>
 <wire x1="50.8" y1="187.96" x2="50.8" y2="182.88" width="0.1524" layer="91"/>
-<pinref part="Y1" gate="Y1" pin="1"/>
+<pinref part="Y1" gate="G$1" pin="1"/>
 <wire x1="50.8" y1="182.88" x2="50.8" y2="180.34" width="0.1524" layer="91"/>
 <wire x1="55.88" y1="182.88" x2="50.8" y2="182.88" width="0.1524" layer="91"/>
@@
 <pinref part="C6" gate="G$1" pin="1"/>
 <wire x1="66.04" y1="180.34" x2="66.04" y2="182.88" width="0.1524" layer="91"/>
-<pinref part="Y1" gate="Y1" pin="2"/>
+<pinref part="Y1" gate="G$1" pin="2"/>
 <wire x1="66.04" y1="182.88" x2="66.04" y2="185.42" width="0.1524" layer="91"/>
 <wire x1="60.96" y1="182.88" x2="66.04" y2="182.88" width="0.1524" layer="91"/>

Commit message: Switched C21 from 0402 to 0603 package
Due to sourcing issues.
Parts:
- C21: device SparkFun-Capacitors:0.1UF-0402T-50V-10%-X7R-WE -> SparkFun-Capacitors:0.1UF-0603-50V-10%-X7R-WE
Changed lines of the file:
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@@
 <grid distance="0.1" unitdist="inch" unit="inch" style="lines" multiple="1" display="no" altdistance="0.01" altunitdist="inch" altunit="inch"/>
 <layers>
-<layer number="1" name="Top" color="4" fill="1" visible="yes" active="no"/>
-<layer number="2" name="Route2" color="1" fill="3" visible="yes" active="no"/>
-<layer number="3" name="Route3" color="4" fill="3" visible="yes" active="no"/>
-<layer number="4" name="Route4" color="1" fill="4" visible="yes" active="no"/>
-<layer number="5" name="Route5" color="4" fill="4" visible="yes" active="no"/>
-<layer number="6" name="Route6" color="1" fill="8" visible="yes" active="no"/>
-<layer number="7" name="Route7" color="4" fill="8" visible="yes" active="no"/>
-<layer number="8" name="Route8" color="1" fill="2" visible="yes" active="no"/>
-<layer number="9" name="Route9" color="4" fill="2" visible="yes" active="no"/>
-<layer number="10" name="Route10" color="1" fill="7" visible="yes" active="no"/>
-<layer number="11" name="Route11" color="4" fill="7" visible="yes" active="no"/>
-<layer number="12" name="Route12" color="1" fill="5" visible="yes" active="no"/>
-<layer number="13" name="Route13" color="4" fill="5" visible="yes" active="no"/>
-<layer number="14" name="Route14" color="1" fill="6" visible="yes" active="no"/>
-<layer number="15" name="Route15" color="4" fill="6" visible="yes" active="no"/>
-<layer number="16" name="Bottom" color="1" fill="1" visible="yes" active="no"/>
-<layer number="17" name="Pads" color="2" fill="1" visible="yes" active="no"/>
-<layer number="18" name="Vias" color="2" fill="1" visible="yes" active="no"/>
-<layer number="19" name="Unrouted" color="6" fill="1" visible="yes" active="no"/>
-<layer number="20" name="Dimension" color="24" fill="1" visible="yes" active="no"/>
-<layer number="21" name="tPlace" color="16" fill="1" visible="yes" active="no"/>
-<layer number="22" name="bPlace" color="14" fill="1" visible="yes" active="no"/>
-<layer number="23" name="tOrigins" color="15" fill="1" visible="yes" active="no"/>
-<layer number="24" name="bOrigins" color="15" fill="1" visible="yes" active="no"/>
-<layer number="25" name="tNames" color="7" fill="1" visible="yes" active="no"/>
-<layer number="26" name="bNames" color="7" fill="1" visible="yes" active="no"/>
-<layer number="27" name="tValues" color="7" fill="1" visible="yes" active="no"/>
-<layer number="28" name="bValues" color="7" fill="1" visible="yes" active="no"/>
+<layer number="1" name="Top" color="4" fill="1" visible="no" active="no"/>
+<layer number="2" name="Route2" color="1" fill="3" visible="no" active="no"/>
+<layer number="3" name="Route3" color="4" fill="3" visible="no" active="no"/>
+<layer number="4" name="Route4" color="1" fill="4" visible="no" active="no"/>
+<layer number="5" name="Route5" color="4" fill="4" visible="no" active="no"/>
+<layer number="6" name="Route6" color="1" fill="8" visible="no" active="no"/>
+<layer number="7" name="Route7" color="4" fill="8" visible="no" active="no"/>
+<layer number="8" name="Route8" color="1" fill="2" visible="no" active="no"/>
+<layer number="9" name="Route9" color="4" fill="2" visible="no" active="no"/>
+<layer number="10" name="Route10" color="1" fill="7" visible="no" active="no"/>
+<layer number="11" name="Route11" color="4" fill="7" visible="no" active="no"/>
+<layer number="12" name="Route12" color="1" fill="5" visible="no" active="no"/>
+<layer number="13" name="Route13" color="4" fill="5" visible="no" active="no"/>
+<layer number="14" name="Route14" color="1" fill="6" visible="no" active="no"/>
+<layer number="15" name="Route15" color="4" fill="6" visible="no" active="no"/>
+<layer number="16" name="Bottom" color="1" fill="1" visible="no" active="no"/>
+<layer number="17" name="Pads" color="2" fill="1" visible="no" active="no"/>
+<layer number="18" name="Vias" color="2" fill="1" visible="no" active="no"/>
+<layer number="19" name="Unrouted" color="6" fill="1" visible="no" active="no"/>
+<layer number="20" name="Dimension" color="24" fill="1" visible="no" active="no"/>
+<layer number="21" name="tPlace" color="16" fill="1" visible="no" active="no"/>
+<layer number="22" name="bPlace" color="14" fill="1" visible="no" active="no"/>
+<layer number="23" name="tOrigins" color="15" fill="1" visible="no" active="no"/>
+<layer number="24" name="bOrigins" color="15" fill="1" visible="no" active="no"/>
+<layer number="25" name="tNames" color="7" fill="1" visible="no" active="no"/>
+<layer number="26" name="bNames" color="7" fill="1" visible="no" active="no"/>
+<layer number="27" name="tValues" color="7" fill="1" visible="no" active="no"/>
+<layer number="28" name="bValues" color="7" fill="1" visible="no" active="no"/>
 <layer number="29" name="tStop" color="7" fill="3" visible="no" active="no"/>
 <layer number="30" name="bStop" color="7" fill="6" visible="no" active="no"/>
@@
 <layer number="35" name="tGlue" color="7" fill="4" visible="no" active="no"/>
 <layer number="36" name="bGlue" color="7" fill="5" visible="no" active="no"/>
-<layer number="37" name="tTest" color="7" fill="1" visible="yes" active="no"/>
-<layer number="38" name="bTest" color="7" fill="1" visible="yes" active="no"/>
+<layer number="37" name="tTest" color="7" fill="1" visible="no" active="no"/>
+<layer number="38" name="bTest" color="7" fill="1" visible="no" active="no"/>
 <layer number="39" name="tKeepout" color="4" fill="11" visible="no" active="no"/>
 <layer number="40" name="bKeepout" color="1" fill="11" visible="no" active="no"/>
@@
 <layer number="44" name="Drills" color="7" fill="1" visible="no" active="no"/>
 <layer number="45" name="Holes" color="7" fill="1" visible="no" active="no"/>
-<layer number="46" name="Milling" color="3" fill="1" visible="yes" active="no"/>
-<layer number="47" name="Measures" color="7" fill="1" visible="yes" active="no"/>
-<layer number="48" name="Document" color="7" fill="1" visible="yes" active="no"/>
-<layer number="49" name="Reference" color="7" fill="1" visible="yes" active="no"/>
-<layer number="50" name="dxf" color="7" fill="1" visible="yes" active="no"/>
-<layer number="51" name="tDocu" color="6" fill="1" visible="yes" active="no"/>
-<layer number="52" name="bDocu" color="7" fill="1" visible="yes" active="no"/>
-<layer number="53" name="tGND_GNDA" color="7" fill="9" visible="yes" active="no"/>
-<layer number="54" name="bGND_GNDA" color="1" fill="9" visible="yes" active="no"/>
-<layer number="56" name="wert" color="7" fill="1" visible="yes" active="no"/>
-<layer number="57" name="tCAD" color="7" fill="1" visible="yes" active="no"/>
-<layer number="58" name="bCAD" color="7" fill="1" visible="yes" active="no"/>
-<layer number="59" name="tCarbon" color="7" fill="1" visible="yes" active="no"/>
-<layer number="60" name="bCarbon" color="7" fill="1" visible="yes" active="no"/>
+<layer number="46" name="Milling" color="3" fill="1" visible="no" active="no"/>
+<layer number="47" name="Measures" color="7" fill="1" visible="no" active="no"/>
+<layer number="48" name="Document" color="7" fill="1" visible="no" active="no"/>
+<layer number="49" name="Reference" color="7" fill="1" visible="no" active="no"/>
+<layer number="50" name="dxf" color="7" fill="1" visible="no" active="no"/>
+<layer number="51" name="tDocu" color="6" fill="1" visible="no" active="no"/>
+<layer number="52" name="bDocu" color="7" fill="1" visible="no" active="no"/>
+<layer number="53" name="tGND_GNDA" color="7" fill="9" visible="no" active="no"/>
+<layer number="54" name="bGND_GNDA" color="1" fill="9" visible="no" active="no"/>
+<layer number="56" name="wert" color="7" fill="1" visible="no" active="no"/>
+<layer number="57" name="tCAD" color="7" fill="1" visible="no" active="no"/>
+<layer number="58" name="bCAD" color="7" fill="1" visible="no" active="no"/>
+<layer number="59" name="tCarbon" color="7" fill="1" visible="no" active="no"/>
+<layer number="60" name="bCarbon" color="7" fill="1" visible="no" active="no"/>
 <layer number="88" name="SimResults" color="9" fill="1" visible="yes" active="yes"/>
 <layer number="89" name="SimProbes" color="9" fill="1" visible="yes" active="yes"/>
@@
 <part name="C20" library="SparkFun-Capacitors" deviceset="1.0NF/1000PF" device="-1206-2KV-10%-X7R-WORTH-ELEKRONIK" value="1.0nF/2kV"/>
 <part name="R23" library="SparkFun-Resistors" deviceset="100OHM" device="-0603-1/10W-1%" value="100Ω"/>
-<part name="C21" library="SparkFun-Capacitors" deviceset="0.1UF" device="-0402T-50V-10%-X7R-WE" value="0.1uF"/>
+<part name="C21" library="SparkFun-Capacitors" deviceset="0.1UF" device="-0603-50V-10%-X7R-WE" value="0.1uF"/>
 <part name="C22" library="SparkFun-Capacitors" deviceset="0.1UF" device="-0603-100V-10%-X7R-WE" value="0.1uF"/>
 <part name="GND14" library="SparkFun-PowerSymbols" deviceset="GND" device=""/>

Commit message: Add Prod_IDs to T1 connectors
updated single and panel brd files
Parts:
- J1: value T1_INDUSTRIAL -> IP20(RJ50)
Changed lines of the file:
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@@
 <part name="C2" library="SparkFun-Capacitors" deviceset="0.22UF" device="-0603-50V-10%" value="0.22uF"/>
 <part name="C1" library="SparkFun-Capacitors" deviceset="0.22UF" device="-0603-50V-10%" value="0.22uF"/>
-<part name="J1" library="ADIN1110" deviceset="T1_INDUSTRIAL_JACK_AH_IP20" device="" value="T1_INDUSTRIAL"/>
+<part name="J1" library="ADIN1110" deviceset="T1_INDUSTRIAL_JACK_AH_IP20" device="" value="IP20(RJ50)"/>
 <part name="SHLD" library="SparkFun-Jumpers" deviceset="JUMPER-SMT_3_1-NC_TRACE" device="_SILK" package3d_urn="urn:adsk.eagle:package:39288/1" value=""/>
 <part name="GND2" library="SparkFun-PowerSymbols" deviceset="GND" device=""/>

Commit message: R3, R4, R5, R6 to in-house PROD_IDs
Note, these values are very slightly different than the ones in the DS sch.
Parts:
- R3, R4: value 5.1Ω -> 4.7; device SparkFun-Resistors:RESISTOR0402T -> SparkFun-Resistors:4.7OHM-0402T-1/16W-1%
- R5, R6: value 10.2Ω -> 10Ω; device SparkFun-Resistors:RESISTOR0402T -> SparkFun-Resistors:10OHM-0402-1/16W-5%
Changed lines of the file:
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@@
 <part name="GND46" library="SparkFun-PowerSymbols" deviceset="GND" device=""/>
 <part name="GND47" library="SparkFun-PowerSymbols" deviceset="GND" device=""/>
-<part name="R5" library="SparkFun-Resistors" deviceset="RESISTOR" device="0402T" value="10.2Ω"/>
-<part name="R6" library="SparkFun-Resistors" deviceset="RESISTOR" device="0402T" value="10.2Ω"/>
-<part name="R4" library="SparkFun-Resistors" deviceset="RESISTOR" device="0402T" value="5.1Ω"/>
-<part name="R3" library="SparkFun-Resistors" deviceset="RESISTOR" device="0402T" value="5.1Ω"/>
+<part name="R5" library="SparkFun-Resistors" deviceset="10OHM" device="-0402-1/16W-5%" value="10Ω"/>
+<part name="R6" library="SparkFun-Resistors" deviceset="10OHM" device="-0402-1/16W-5%" value="10Ω"/>
+<part name="R4" library="SparkFun-Resistors" deviceset="4.7OHM" device="-0402T-1/16W-1%" value="4.7"/>
+<part name="R3" library="SparkFun-Resistors" deviceset="4.7OHM" device="-0402T-1/16W-1%" value="4.7"/>
 <part name="C2" library="SparkFun-Capacitors" deviceset="0.22UF" device="-0603-50V-10%" value="0.22uF"/>
 <part name="C1" library="SparkFun-Capacitors" deviceset="0.22UF" device="-0603-50V-10%" value="0.22uF"/>

Commit message: TVS diode placement and more
-Moved TVS diodes to "IC" side of DA-/DA+ DC coupling caps
-Added debounce to reset button
-Routed through pads 5 and 6 on TVS diode package.
-Added R29 to avoid damaging GPIO if set to output low and button pressed
-Added R26 to mosfet gate control line to avoid potential overvoltage/ringing
-Re-arranged caps so smalled value decoupling caps are closest to pins on IC.
-moved to "v10" in brd and sch
-C22 changed to 470nF to improove droop performance
Parts:
- added C23: 0.1uF, SparkFun-Capacitors:0.1UF-0402T-16V-10%-X7R-WE
- added R26: 100, SparkFun-Resistors:100OHM-0603-1/10W-1%
- added R27: 10k, SparkFun-Resistors:10KOHM-0603-1/10W-1%
- added R28: 100k, SparkFun-Resistors:100KOHM-0402T-1/16W-1%
- added R29: 100Ω, SparkFun-Resistors:100OHM-0603-1/10W-1%
- C22: value 0.1uF -> 470nF; device SparkFun-Capacitors:0.1UF-0603-100V-10%-X7R-WE -> SparkFun-Capacitors:470NF-0603-10V-10%-X5R
- R3, R4: value 4.7 -> 5.1k; device SparkFun-Resistors:4.7OHM-0402T-1/16W-1% -> SparkFun-Resistors:5.1KOHM-0402T-1/16W-1%
- R5, R6: value 10Ω -> 10.2k; device SparkFun-Resistors:10OHM-0402-1/16W-5% -> SparkFun-Resistors:10.2KOHM-0402-1/16W-1%
Connections:
- new net N$10: Q1.D, R26.1
- new net N$13: C23.1, R27.1, U1.!RESET!
- new net N$15: R27.2, R28.1, R29.2, S1.2
- net !RESET!: now also R29.1; no longer S1.2, U1.!RESET!
- net 3.3V: now also R28.2
- net GND: now also C23.2
- net N$11: now also R26.2; no longer Q1.D
- net N$24: now also U4.2
- net N$31: now also U4.1
- net N$32: no longer U4.2
- net N$34: no longer U4.1
Other:
- note removed: "*reset has internal pullup"
- moved on the sheet: C1, C10, C11, C12, C13, C14, C15, C16, C17, C18, C19, C2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
